File: summer project 1.1.kicad_pcb (KiCad board)
At the start: 2 copper layers, 47.4 x 23.2 mm, 11 parts, among them J1 Conn_01x02_Socket, J2 Conn_01x02_Socket, J3 Screw_Terminal_01x02, Q1 NMOS, Q2 NMOS, U1 LM5050-1_mod2, U2 LM5050-1_mod2

Commit message: Routing Completed
Parts:
- moved Q1 2.14 mm to (131.2, 77.2)
- moved U2 2.14 mm to (144.4, 85.9)
- moved C1 2.14 mm to (137.5, 84.5)
- moved J2 2.14 mm to (137.5, 91.9)
- moved J3 2.14 mm to (160.0, 79.5)
- moved R1 2.14 mm to (137.5, 80.2)
- moved C2 2.14 mm to (150.5, 85.6)
- moved J1 2.14 mm to (122.2, 77.4)
- moved Q2 2.14 mm to (144.5, 77.3)
- moved R2 2.14 mm to (150.3, 81.6)
- moved U1 2.14 mm to (131.2, 86.5)
Routing:
- net VCC (Vout): track 0.80 -> 48.4 mm, vias 0 -> 4
- net Net-(U2-VS): track 0.00 -> 25.7 mm
- net Net-(Q1-G): track 4.07 -> 23.2 mm
- net MAIN BATT: track 0.00 -> 18.9 mm, vias 0 -> 2
- net Net-(U1-VS): track 0.18 -> 13.2 mm
- net BACKUP BATT: track 0.00 -> 12.3 mm
- net Net-(Q2-G): track 0.14 -> 9.00 mm
- net GND: vias 0 -> 72
- added copper zone on F.Cu, net BACKUP BATT
- added copper zone on B.Cu, net GND
- added copper zone on F.Cu, net GND
- added copper zone on F.Cu, net MAIN BATT
Other:
- board text added: "LM5050 Redundancy Circuit"
