File: summer project 1.1.kicad_sch (KiCad schematic)
At the start: 1 part, among them U3 LM5050-1_mod2

Commit message: Schematic Design Completed
Parts:
- added C3, C4: 0.1u, Capacitor_SMD:C_0603_1608Metric, symbol Device:C_Small
- added J4, J5: Conn_01x02_Socket, Connector_AMASS:AMASS_XT30U-F_1x02_P5.0mm_Vertical, symbol Connector:Conn_01x02_Socket
- added J6: Screw_Terminal_01x02, TerminalBlock_Phoenix:TerminalBlock_Phoenix_MKDS-3-2-5.08_1x02_P5.08mm_Horizontal, symbol Connector:Screw_Terminal_01x02
- added Q3, Q4: NMOS, Package_TO_SOT_SMD:TO-252-3_TabPin2, symbol Simulation_SPICE:NMOS
- added R3, R4: 100, Resistor_SMD:R_0603_1608Metric, symbol Device:R_Small
- added U4: LM5050-1_mod2, Package_TO_SOT_SMD:TSOT-23-6, symbol smp 1:LM5050-1_mod2
Connections:
- net at U3.1 (VS): now also C3.2, R3.1
- net GND: now reaches U3.2 (GND)
- net GND: now also U3.3 (OFF), C3.1, C4.1, J4.1 (Pin_1), J5.1 (Pin_1), J6.2 (Pin_2), U4.2 (GND), U4.3 (OFF)
- net MAIN BATT: now reaches U3.4 (IN)
- net MAIN BATT: now also J5.2 (Pin_2), Q3.3 (S)
- net at U3.5 (GATE): now also Q3.2 (G)
- net VCC (Vout): now reaches U3.6 (OUT)
- net VCC (Vout): now also J6.1 (Pin_1), Q3.1 (D), Q4.1 (D), R3.2, R4.2, U4.6 (OUT)
- new net: C4.2, R4.1, U4.1 (VS)
- new net: Q4.2 (G), U4.5 (GATE)
- new net BACKUP BATT: J4.2 (Pin_2), Q4.3 (S), U4.4 (IN)

Commit message: Pages Titled
Other:
- title: (none) -> LM5050 REDUNDANCY POWER CIRCUIT-AUV
Changed lines of the file:
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@@
 	(generator_version "9.0")
 	(paper "A4")
+	(title_block
+		(title "LM5050 REDUNDANCY POWER CIRCUIT-AUV")
+		(date "03/06/2026")
+	)
 	(junction
 		(at 168.91 115.57)

Commit message: symbol design
Parts:
- removed U3, U4: LM5050-1_mod2, Package_TO_SOT_SMD:TSOT-23-6, symbol smp 1:LM5050-1_mod2
- added U1, U2: LM5050-1_mod2, Package_TO_SOT_SMD:TSOT-23-6, symbol smp1:LM5050-1_mod2
Connections:
- net BACKUP BATT: now also U2.4 (IN)
- net GND: now also U1.2 (GND), U1.3 (OFF), U2.2 (GND), U2.3 (OFF)
- net MAIN BATT: now also U1.4 (IN)
- net VCC (Vout): now also U1.6 (OUT), U2.6 (OUT)
- net at C3.2, R3.1: now also U1.1 (VS)
- net at C4.2, R4.1: now also U2.1 (VS)
- net at Q4.2 (G): now also U2.5 (GATE)
- net at Q3.2 (G): now also U1.5 (GATE)
Changed lines of the file:
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@@
-	)
-	(symbol
-		(lib_id "smp 1:LM5050-1_mod2")
-		(at 138.43 114.3 90)
-		(unit 1)
-		(exclude_from_sim no)
-		(in_bom yes)
-		(on_board yes)
-		(dnp no)
-		(property "Reference" "U4"
-			(at 140.97 117.094 90)
-			(effects
-				(font
-					(size 1.27 1.27)
-				)
-			)
-		)
-		(property "Value" "LM5050-1_mod2"
-			(at 141.732 118.618 90)
-			(effects
-				(font
-					(size 0.635 0.635)
-				)
-			)
-		)
-		(property "Footprint" "Package_TO_SOT_SMD:TSOT-23-6"
-			(at 147.32 97.79 0)
-			(effects
-				(font
-					(size 1.27 1.27)
-				)
-				(hide yes)
-			)
-		)
-		(property "Datasheet" "http://www.ti.com/lit/ds/symlink/lm5050-1-q1.pdf"
-			(at 139.7 86.36 0)
-			(effects
-				(font
-					(size 1.27 1.27)
-				)
-				(hide yes)
-			)
-		)
-		(property "Description" "High side OR-ing FET controller, 5V to 75V operation, TSOT-23-6"
-			(at 138.43 114.3 0)
-			(effects
-				(font
-					(size 1.27 1.27)
-				)
-				(hide yes)
-			)
-		)
-		(pin "5"
-		)
-		(pin "1"
-		)
-		(pin "6"
-		)
-		(pin "4"
-		)
-		(pin "2"
-		)
-		(pin "3"
-		)
-		(instances
-			(project "summer project 1.1"
-				(path "/19e44473-05a8-487a-9fcb-12427ac5e96b"
-					(reference "U4")
-					(unit 1)
-				)
-			)
-		)
-	)
-	(symbol
-		(lib_id "smp 1:LM5050-1_mod2")
-		(at 137.16 72.39 90)
-		(unit 1)
-		(exclude_from_sim no)
-		(in_bom yes)
-		(on_board yes)
-		(dnp no)
-		(property "Reference" "U3"
-			(at 139.7 75.184 90)
-			(effects
-				(font
-					(size 1.27 1.27)
-				)
-			)
-		)
-		(property "Value" "LM5050-1_mod2"
-			(at 140.462 76.708 90)
-			(effects
-				(font
-					(size 0.635 0.635)
-				)
-			)
-		)
-		(property "Footprint" "Package_TO_SOT_SMD:TSOT-23-6"
-			(at 146.05 55.88 0)
-			(effects
-				(font
-					(size 1.27 1.27)
-				)
-				(hide yes)
-			)
-		)
-		(property "Datasheet" "http://www.ti.com/lit/ds/symlink/lm5050-1-q1.pdf"
-			(at 138.43 44.45 0)
-			(effects
-				(font
-					(size 1.27 1.27)
-				)
-				(hide yes)
-			)
-		)
-		(property "Description" "High side OR-ing FET controller, 5V to 75V operation, TSOT-23-6"
-			(at 137.16 72.39 0)
-			(effects
-				(font
-					(size 1.27 1.27)
-				)
-				(hide yes)
-			)
-		)
-		(pin "5"
-		)
-		(pin "1"
-		)
-		(pin "6"
-		)
-		(pin "4"
-		)
-		(pin "2"
-		)
-		(pin "3"
-		)
-		(instances
-			(project "summer project 1.1"
-				(path "/19e44473-05a8-487a-9fcb-12427ac5e96b"
-					(reference "U3")
-					(unit 1)
-				)
-			)
-		)
 	)
 	(symbol
@@
 	)
 	(symbol
+		(lib_id "smp1:LM5050-1_mod2")
+		(at 138.43 114.3 90)
+		(unit 1)
+		(exclude_from_sim no)
+		(in_bom yes)
+		(on_board yes)
+		(dnp no)
+		(fields_autoplaced yes)
+		(property "Reference" "U2"
+			(at 156.21 110.1246 90)
+			(effects
+				(font
+					(size 1.27 1.27)
+				)
+			)
+		)
+		(property "Value" "LM5050-1_mod2"
+			(at 156.21 112.6646 90)
+			(effects
+				(font
+					(size 1.27 1.27)
+				)
+			)
+		)
+		(property "Footprint" "Package_TO_SOT_SMD:TSOT-23-6"
+			(at 147.32 97.79 0)
+			(effects
+				(font
+					(size 1.27 1.27)
+				)
+				(hide yes)
+			)
+		)
+		(property "Datasheet" "http://www.ti.com/lit/ds/symlink/lm5050-1-q1.pdf"
+			(at 139.7 86.36 0)
+			(effects
+				(font
+					(size 1.27 1.27)
+				)
+				(hide yes)
+			)
+		)
+		(property "Description" "High side OR-ing FET controller, 5V to 75V operation, TSOT-23-6"
+			(at 138.43 114.3 0)
+			(effects
+				(font
+					(size 1.27 1.27)
+				)
+				(hide yes)
+			)
+		)
+		(pin "6"
+		)
+		(pin "5"
+		)
+		(pin "2"
+		)
+		(pin "1"
+		)
+		(pin "3"
+		)
+		(pin "4"
+		)
+		(instances
+			(project "summer project 1.1"
+				(path "/19e44473-05a8-487a-9fcb-12427ac5e96b"
+					(reference "U2")
+					(unit 1)
+				)
+			)
+		)
+	)
+	(symbol
 		(lib_id "power:GND")
 		(at 175.26 64.77 0)
@@
 					(unit 1)
 				)
+			)
+		)
+	)
+	(symbol
+		(lib_id "smp1:LM5050-1_mod2")
+		(at 137.16 72.39 90)
+		(unit 1)
+		(exclude_from_sim no)
+		(in_bom yes)
+		(on_board yes)
+		(dnp no)
+		(fields_autoplaced yes)
+		(property "Reference" "U1"
+			(at 154.94 68.2146 90)
+			(effects
+				(font
+					(size 1.27 1.27)
+				)
+			)
+		)
+		(property "Value" "LM5050-1_mod2"
+			(at 154.94 70.7546 90)
+			(effects
+				(font
+					(size 1.27 1.27)
+				)
+			)
+		)
+		(property "Footprint" "Package_TO_SOT_SMD:TSOT-23-6"
+			(at 146.05 55.88 0)
+			(effects
+				(font
+					(size 1.27 1.27)
+				)
+				(hide yes)
+			)
+		)
+		(property "Datasheet" "http://www.ti.com/lit/ds/symlink/lm5050-1-q1.pdf"
+			(at 138.43 44.45 0)
+			(effects
+				(font
+					(size 1.27 1.27)
+				)
+				(hide yes)
+			)
+		)
+		(property "Description" "High side OR-ing FET controller, 5V to 75V operation, TSOT-23-6"
+			(at 137.16 72.39 0)
+			(effects
+				(font
+					(size 1.27 1.27)
+				)
+				(hide yes)
+			)
+		)
+		(pin "6"
+		)
+		(pin "5"
+		)
+		(pin "2"
+		)
+		(pin "1"
+		)
+		(pin "3"
+		)
+		(pin "4"
+		)
+		(instances
+			(project ""
+				(path "/19e44473-05a8-487a-9fcb-12427ac5e96b"
+					(reference "U1")
+					(unit 1)
+				)
